File: Compact2Hand/DholydaiComp/DholydaiComp.kicad_pcb (KiCad board)
At the start: 2 copper layers, 304.8 x 136 mm, 175 parts, among them SW1 SW_Push, SW10 SW_Push, SW11 SW_Push, SW12 SW_Push, SW13 SW_Push, SW14 SW_Push, SW15 SW_Push, SW16 SW_Push, SW17 SW_Push, SW18 SW_Push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

Commit message: Add files via upload
Other:
- outline, holes or cut-outs redrawn
- board text added: "Quixotic Keyboards, LLC Post-Mechanical Compact 27 Jun 2024 v1.11 Dholydai"
- board text removed: "Quixotic Keyboards, LLC Post-Mech Compact 140 Apr 2024 v1.1 Dholydai"
